File: hardware/controller/power.kicad_sch (KiCad schematic)
At the start: 16 parts, among them J11 Barrel_Jack, J7 Conn_01x04_Pin, J8 Conn_01x04_Pin, U7 MPM3606AGQV-P, U8 LM73100RPWR, U9 LM73100RPWR

Commit message: Update some LCSC numbers
Parts:
- U7: LCSC (none) -> C7305220
Changed lines of the file:
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@@
+				)
+			)
+			(project "power"
+				(path "/f3545cb4-b0c7-49de-9654-d098df7deee8"
+					(reference "TP?")
+					(unit 1)
 				)
 			)
@@
 				)
 			)
+			(project "power"
+				(path "/f3545cb4-b0c7-49de-9654-d098df7deee8"
+					(reference "#PWR?")
+					(unit 1)
+				)
+			)
 		)
 	)
@@
 				)
 			)
+			(project "power"
+				(path "/f3545cb4-b0c7-49de-9654-d098df7deee8"
+					(reference "#PWR?")
+					(unit 1)
+				)
+			)
 		)
 	)
@@
 				)
 			)
+			(project "power"
+				(path "/f3545cb4-b0c7-49de-9654-d098df7deee8"
+					(reference "#PWR?")
+					(unit 1)
+				)
+			)
 		)
 	)
@@
 				)
 			)
+			(project "power"
+				(path "/f3545cb4-b0c7-49de-9654-d098df7deee8"
+					(reference "#PWR?")
+					(unit 1)
+				)
+			)
 		)
 	)
@@
 				)
 			)
+			(project "power"
+				(path "/f3545cb4-b0c7-49de-9654-d098df7deee8"
+					(reference "U?")
+					(unit 1)
+				)
+			)
 		)
 	)
@@
 				)
 			)
+			(project "power"
+				(path "/f3545cb4-b0c7-49de-9654-d098df7deee8"
+					(reference "#PWR?")
+					(unit 1)
+				)
+			)
 		)
 	)
@@
 				)
 			)
+			(project "power"
+				(path "/f3545cb4-b0c7-49de-9654-d098df7deee8"
+					(reference "#PWR?")
+					(unit 1)
+				)
+			)
 		)
 	)
@@
 				)
 			)
+			(project "power"
+				(path "/f3545cb4-b0c7-49de-9654-d098df7deee8"
+					(reference "#PWR?")
+					(unit 1)
+				)
+			)
 		)
 	)
@@
 				)
 			)
+			(project "power"
+				(path "/f3545cb4-b0c7-49de-9654-d098df7deee8"
+					(reference "#PWR?")
+					(unit 1)
+				)
+			)
 		)
 	)
@@
 				)
 			)
+			(project "power"
+				(path "/f3545cb4-b0c7-49de-9654-d098df7deee8"
+					(reference "TP?")
+					(unit 1)
+				)
+			)
 		)
 	)
@@
 				)
 			)
+			(project "power"
+				(path "/f3545cb4-b0c7-49de-9654-d098df7deee8"
+					(reference "R?")
+					(unit 1)
+				)
+			)
 		)
 	)
@@
 				)
 			)
+			(project "power"
+				(path "/f3545cb4-b0c7-49de-9654-d098df7deee8"
+					(reference "#PWR?")
+					(unit 1)
+				)
+			)
 		)
 	)
@@
 				)
 			)
+			(project "power"
+				(path "/f3545cb4-b0c7-49de-9654-d098df7deee8"
+					(reference "C?")
+					(unit 1)
+				)
+			)
 		)
 	)
@@
 				)
 			)
+			(project "power"
+				(path "/f3545cb4-b0c7-49de-9654-d098df7deee8"
+					(reference "R?")
+					(unit 1)
+				)
+			)
 		)
 	)
@@
 				(path "/3ee12552-bbaf-4643-8241-99077a41063f/dc443349-7fb4-42c6-a18e-09a219bb9ecd"
 					(reference "#PWR028")
+					(unit 1)
+				)
+			)
+			(project "power"
+				(path "/f3545cb4-b0c7-49de-9654-d098df7deee8"
+					(reference "#PWR?")
 					(unit 1)
 				)
@@
 				)
 			)
+			(project "power"
+				(path "/f3545cb4-b0c7-49de-9654-d098df7deee8"
+					(reference "J?")
+					(unit 1)
+				)
+			)
 		)
 	)
@@
 				)
 			)
+			(project "power"
+				(path "/f3545cb4-b0c7-49de-9654-d098df7deee8"
+					(reference "#PWR?")
+					(unit 1)
+				)
+			)
 		)
 	)
@@
 				)
 			)
+			(project "power"
+				(path "/f3545cb4-b0c7-49de-9654-d098df7deee8"
+					(reference "#PWR?")
+					(unit 1)
+				)
+			)
 		)
 	)
@@
 				)
 			)
+			(project "power"
+				(path "/f3545cb4-b0c7-49de-9654-d098df7deee8"
+					(reference "C?")
+					(unit 1)
+				)
+			)
 		)
 	)
@@
 				)
 			)
+			(project "power"
+				(path "/f3545cb4-b0c7-49de-9654-d098df7deee8"
+					(reference "#PWR?")
+					(unit 1)
+				)
+			)
 		)
 	)
@@
 				)
 			)
+			(project "power"
+				(path "/f3545cb4-b0c7-49de-9654-d098df7deee8"
+					(reference "#PWR?")
+					(unit 1)
+				)
+			)
 		)
 	)
@@
 				)
 			)
+			(project "power"
+				(path "/f3545cb4-b0c7-49de-9654-d098df7deee8"
+					(reference "J?")
+					(unit 1)
+				)
+			)
 		)
 	)
@@
 				)
 			)
+			(project "power"
+				(path "/f3545cb4-b0c7-49de-9654-d098df7deee8"
+					(reference "C?")
+					(unit 1)
+				)
+			)
 		)
 	)
@@
 				)
 			)
+			(project "power"
+				(path "/f3545cb4-b0c7-49de-9654-d098df7deee8"
+					(reference "TP?")
+					(unit 1)
+				)
+			)
 		)
 	)
@@
 				)
 			)
+			(project "power"
+				(path "/f3545cb4-b0c7-49de-9654-d098df7deee8"
+					(reference "#PWR?")
+					(unit 1)
+				)
+			)
 		)
 	)
@@
 				)
 			)
+			(project "power"
+				(path "/f3545cb4-b0c7-49de-9654-d098df7deee8"
+					(reference "#PWR?")
+					(unit 1)
+				)
+			)
 		)
 	)
@@
 				)
 			)
+			(project "power"
+				(path "/f3545cb4-b0c7-49de-9654-d098df7deee8"
+					(reference "#PWR?")
+					(unit 1)
+				)
+			)
 		)
 	)
@@
 				)
 			)
+			(project "power"
+				(path "/f3545cb4-b0c7-49de-9654-d098df7deee8"
+					(reference "#PWR?")
+					(unit 1)
+				)
+			)
 		)
 	)
@@
 				)
 			)
+			(project "power"
+				(path "/f3545cb4-b0c7-49de-9654-d098df7deee8"
+					(reference "U?")
+					(unit 1)
+				)
+			)
 		)
 	)
@@
 				(path "/3ee12552-bbaf-4643-8241-99077a41063f/dc443349-7fb4-42c6-a18e-09a219bb9ecd"
 					(reference "#PWR030")
+					(unit 1)
+				)
+			)
+			(project "power"
+				(path "/f3545cb4-b0c7-49de-9654-d098df7deee8"
+					(reference "#PWR?")
 					(unit 1)
 				)
@@
 				)
 			)
+			(project "power"
+				(path "/f3545cb4-b0c7-49de-9654-d098df7deee8"
+					(reference "J?")
+					(unit 1)
+				)
+			)
 		)
 	)
@@
 				)
 			)
+			(project "power"
+				(path "/f3545cb4-b0c7-49de-9654-d098df7deee8"
+					(reference "#PWR?")
+					(unit 1)
+				)
+			)
 		)
 	)
@@
 				)
 			)
+			(project "power"
+				(path "/f3545cb4-b0c7-49de-9654-d098df7deee8"
+					(reference "R?")
+					(unit 1)
+				)
+			)
 		)
 	)
@@
 			)
 		)
+		(property "LCSC" "C7305220"
+			(at 78.74 113.03 0)
+			(effects
+				(font
+					(size 1.27 1.27)
+				)
+				(hide yes)
+			)
+		)
 		(pin "16"
 		)
@@
 				(path "/3ee12552-bbaf-4643-8241-99077a41063f/dc443349-7fb4-42c6-a18e-09a219bb9ecd"
 					(reference "U7")
+					(unit 1)
+				)
+			)
+			(project "power"
+				(path "/f3545cb4-b0c7-49de-9654-d098df7deee8"
+					(reference "U?")
 					(unit 1)
 				)
@@
 				)
 			)
+			(project "power"
+				(path "/f3545cb4-b0c7-49de-9654-d098df7deee8"
+					(reference "R?")
+					(unit 1)
+				)
+			)
 		)
 	)
@@
 				)
 			)
-		)
-	)
+			(project "power"
+				(path "/f3545cb4-b0c7-49de-9654-d098df7deee8"
+					(reference "#PWR?")
+					(unit 1)
+				)
+			)
+		)
+	)
+	(sheet_instances
+		(path "/"
+			(page "1")
+		)
+	)
+	(embedded_fonts no)
 )
