File: hardware/controller/mcu.kicad_sch (KiCad schematic)
At the start: 21 parts, among them J12 USB_C_Receptacle_USB2.0_14P, J5 Screw_Terminal_01x02, J6 Screw_Terminal_01x02, U1 ESP32-C3-MINI-1, U6 TPS1H200AQDGNRQ1

Commit message: Update some LCSC numbers
Parts:
- U1: LCSC C2934569 -> C2838502
Changed lines of the file:
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@@
 			)
 		)
-		(property "LCSC" "C2934569"
+		(property "LCSC" "C2838502"
 			(at 146.05 92.71 0)
 			(effects

Commit message: Update LED LCSC
Parts:
- D1: LCSC C114586 -> C2874885
Changed lines of the file:
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@@
 			)
 		)
-		(property "LCSC" "C114586"
+		(property "LCSC" "C2874885"
 			(at 241.3 111.76 0)
 			(effects

Commit message: Add serial number box
Parts:
- U6: FT Rotation Offset (none) -> -90
Changed lines of the file:
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@@
+			)
+		)
+		(property "FT Rotation Offset" "-90"
+			(at 80.01 142.24 0)
+			(effects
+				(font
+					(size 1.27 1.27)
+				)
+				(hide yes)
 			)
 		)

Commit message: Update component position offsets for JLC
Parts:
- J12: FT Position Offset (none) -> 0,1.3335
- U1: FT Position Offset (none) -> 0,-2.7305
Changed lines of the file:
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@@
 			)
 		)
-		(property "Field6" ""
+		(property "FT Position Offset" "0,1.3335"
 			(at 251.46 49.53 0)
 			(effects
@@
 			(at 146.05 92.71 0)
 			(effects
+				(font
+					(size 1.27 1.27)
+				)
+				(hide yes)
+			)
+		)
+		(property "FT Position Offset" "0,-2.7305"
+			(at 146.05 92.71 0)
+			(effects
